Commit message: Configuring the RGB-D Camera
RGB camera exchanged by RGB-D camera by definining:
- new joint
- new link
- world update
- library exchange  (libgazebo_ros_camera.so to libgazebo_ros_openni_kinect.so)

File: my_robot/urdf/my_robot.xacro (robot description, xacro)
@@ -24,4 +24,10 @@
     <dynamics damping="1.0" friction="1.0"/>
   </joint>
+  <joint type="fixed" name="camera_optical_joint">
+    <origin xyz="0 0 0" rpy="-1.5707 0 -1.5707"/>
+    <parent link="camera_link"/>
+    <child link="camera_link_optical"/>
+  </joint>
+  <link name="camera_link_optical"></link>
   <joint type="fixed" name="camera_joint">
     <origin xyz="0.225 0 0" rpy="0 0 0"/>
@@ -136,4 +142,6 @@
     </visual>
 </link>
+<link name="camera_link_optical">
+</link>
 <link name='camera'>
     <pose>0 0 0 0 0 0</pose>

Commit message: Creating launch files for mapping and locatization.
RTAB-Map Localization has been added togeather with some fixes with camera configuration.

File: my_robot/urdf/my_robot.xacro (robot description, xacro)
@@ -24,10 +24,4 @@
     <dynamics damping="1.0" friction="1.0"/>
   </joint>
-  <joint type="fixed" name="camera_optical_joint">
-    <origin xyz="0 0 0" rpy="-1.5707 0 -1.5707"/>
-    <parent link="camera_link"/>
-    <child link="camera_link_optical"/>
-  </joint>
-  <link name="camera_link_optical"></link>
   <joint type="fixed" name="camera_joint">
     <origin xyz="0.225 0 0" rpy="0 0 0"/>
@@ -142,6 +136,4 @@
     </visual>
 </link>
-<link name="camera_link_optical">
-</link>
 <link name='camera'>
     <pose>0 0 0 0 0 0</pose>
